Commit message: cleaned up urdf

File: src/meshes/TriPed.urdf (robot description, URDF)
Before this commit: robot triped, 14 links, 13 joints
Links:
- removed link base_link
Joints:
- removed joint base_to_chassis

Commit message: cleaned up code, added docstrings

File: src/meshes/TriPed.urdf (robot description, URDF)
Before this commit: robot triped, 13 links, 12 joints
Joints:
- joint leg_0_LCSX: limit lower=-1.57079632679 upper=1.57079632679 effort=1000.0 velocity=0.5 -> lower=-0.523599 upper=0.523599 effort=1000.0 velocity=0.5
- joint leg_0_LCSY: limit lower=-1.57079632679 upper=1.57079632679 effort=1000.0 velocity=0.5 -> lower=-0.523599 upper=0.523599 effort=1000.0 velocity=0.5
- joint leg_0_LCSZ: limit lower=-1.57079632679 upper=1.57079632679 effort=1000.0 velocity=0.5 -> lower=-0.523599 upper=0.523599 effort=1000.0 velocity=0.5
- joint leg_1_LCSX: limit lower=-1.57079632679 upper=1.57079632679 effort=1000.0 velocity=0.5 -> lower=-0.523599 upper=0.523599 effort=1000.0 velocity=0.5
- joint leg_1_LCSY: limit lower=-1.57079632679 upper=1.57079632679 effort=1000.0 velocity=0.5 -> lower=-0.523599 upper=0.523599 effort=1000.0 velocity=0.5
- joint leg_1_LCSZ: limit lower=-1.57079632679 upper=1.57079632679 effort=1000.0 velocity=0.5 -> lower=-0.523599 upper=0.523599 effort=1000.0 velocity=0.5
- joint leg_2_LCSX: limit lower=-1.57079632679 upper=1.57079632679 effort=1000.0 velocity=0.5 -> lower=-0.523599 upper=0.523599 effort=1000.0 velocity=0.5
- joint leg_2_LCSY: limit lower=-1.57079632679 upper=1.57079632679 effort=1000.0 velocity=0.5 -> lower=-0.523599 upper=0.523599 effort=1000.0 velocity=0.5
- joint leg_2_LCSZ: limit lower=-1.57079632679 upper=1.57079632679 effort=1000.0 velocity=0.5 -> lower=-0.523599 upper=0.523599 effort=1000.0 velocity=0.5

Commit message: made collision meshes congruent to matlab simulation

File: src/meshes/TriPed.urdf (robot description, URDF)
Before this commit: robot triped, 13 links, 12 joints
Links:
- link leg_0_drive_module: geometry visual mesh filename=drive_module.stl scale=0.001 0.001 0.001
- link leg_0_open: geometry collision sphere radius=0.03; visual mesh filename=leg_linear.stl scale=0.001 0.001 0.001
- link leg_1_drive_module: geometry visual mesh filename=drive_module.stl scale=0.001 0.001 0.001
- link leg_1_open: geometry collision sphere radius=0.03; visual mesh filename=leg_linear.stl scale=0.001 0.001 0.001
- link leg_2_drive_module: geometry visual mesh filename=drive_module.stl scale=0.001 0.001 0.001
- link leg_2_open: geometry collision sphere radius=0.03; visual mesh filename=leg_linear.stl scale=0.001 0.001 0.001

Commit message: added inertia to model

File: src/meshes/TriPed.urdf (robot description, URDF)
Before this commit: robot triped, 13 links, 12 joints
Links:
- link chassis: mass None -> 10.414
- link leg_0_drive_module: mass None -> 1.908
- link leg_0_open: mass None -> 0.503
- link leg_0_rotX: mass None -> 0
- link leg_0_rotY: mass None -> 0
- link leg_1_drive_module: mass None -> 1.908
- link leg_1_open: mass None -> 0.503
- link leg_1_rotX: mass None -> 0
- link leg_1_rotY: mass None -> 0
- link leg_2_drive_module: mass None -> 1.908
- link leg_2_open: mass None -> 0.503
- link leg_2_rotX: mass None -> 0
- link leg_2_rotY: mass None -> 0
