Commit message: added coupling rods to urdf

File: src/triped_sim/robot_descriptions/triped.urdf (robot description, URDF)
Before this commit: robot triped, 19 links, 18 joints
Links:
- added link leg_0_coupling_rod_left; visual mesh filename=coupling_rod.stl scale=0.001 0.001 0.001
- added link leg_0_coupling_rod_right; visual mesh filename=coupling_rod.stl scale=0.001 0.001 0.001
- added link leg_0_rotX_coupling_left, mass 0
- added link leg_0_rotX_coupling_right, mass 0
- added link leg_0_rotY_coupling_left, mass 0
- added link leg_0_rotY_coupling_right, mass 0
- added link leg_1_coupling_rod_left; visual mesh filename=coupling_rod.stl scale=0.001 0.001 0.001
- added link leg_1_coupling_rod_right; visual mesh filename=coupling_rod.stl scale=0.001 0.001 0.001
- added link leg_1_rotX_coupling_left, mass 0
- added link leg_1_rotX_coupling_right, mass 0
- added link leg_1_rotY_coupling_left, mass 0
- added link leg_1_rotY_coupling_right, mass 0
- added link leg_2_coupling_rod_left; visual mesh filename=coupling_rod.stl scale=0.001 0.001 0.001
- added link leg_2_coupling_rod_right; visual mesh filename=coupling_rod.stl scale=0.001 0.001 0.001
- added link leg_2_rotX_coupling_left, mass 0
- added link leg_2_rotX_coupling_right, mass 0
- added link leg_2_rotY_coupling_left, mass 0
- added link leg_2_rotY_coupling_right, mass 0
Joints:
- added joint leg_0_LCSX_coupling_left: type continuous, parent leg_0_left, child leg_0_rotX_coupling_left, origin xyz=0.085 0 -0.0145 rpy=0.0 0.0 0, axis 1.0 0.0 0.0
- added joint leg_0_LCSX_coupling_right: type continuous, parent leg_0_right, child leg_0_rotX_coupling_right, origin xyz=0.085 0 -0.0145 rpy=0.0 0.0 0, axis 1.0 0.0 0.0
- added joint leg_0_LCSY_coupling_left: type continuous, parent leg_0_rotX_coupling_left, child leg_0_rotY_coupling_left, axis 0.0 1.0 0.0
- added joint leg_0_LCSY_coupling_right: type continuous, parent leg_0_rotX_coupling_right, child leg_0_rotY_coupling_right, axis 0.0 1.0 0.0
- added joint leg_0_LCSZ_coupling_left: type continuous, parent leg_0_rotY_coupling_left, child leg_0_coupling_rod_left, axis 0.0 0.0 1.0
- added joint leg_0_LCSZ_coupling_right: type continuous, parent leg_0_rotY_coupling_right, child leg_0_coupling_rod_right, axis 0.0 0.0 1.0
- added joint leg_1_LCSX_coupling_left: type continuous, parent leg_1_left, child leg_1_rotX_coupling_left, origin xyz=0.085 0 -0.0145 rpy=0.0 0.0 0, axis 1.0 0.0 0.0
- added joint leg_1_LCSX_coupling_right: type continuous, parent leg_1_right, child leg_1_rotX_coupling_right, origin xyz=0.085 0 -0.0145 rpy=0.0 0.0 0, axis 1.0 0.0 0.0
- added joint leg_1_LCSY_coupling_left: type continuous, parent leg_1_rotX_coupling_left, child leg_1_rotY_coupling_left, axis 0.0 1.0 0.0
- added joint leg_1_LCSY_coupling_right: type continuous, parent leg_1_rotX_coupling_right, child leg_1_rotY_coupling_right, axis 0.0 1.0 0.0
- added joint leg_1_LCSZ_coupling_left: type continuous, parent leg_1_rotY_coupling_left, child leg_1_coupling_rod_left, axis 0.0 0.0 1.0
- added joint leg_1_LCSZ_coupling_right: type continuous, parent leg_1_rotY_coupling_right, child leg_1_coupling_rod_right, axis 0.0 0.0 1.0
- added joint leg_2_LCSX_coupling_left: type continuous, parent leg_1_left, child leg_2_rotX_coupling_left, origin xyz=0.085 0 -0.0145 rpy=0.0 0.0 0, axis 1.0 0.0 0.0
- added joint leg_2_LCSX_coupling_right: type continuous, parent leg_1_right, child leg_2_rotX_coupling_right, origin xyz=0.085 0 -0.0145 rpy=0.0 0.0 0, axis 1.0 0.0 0.0
- added joint leg_2_LCSY_coupling_left: type continuous, parent leg_2_rotX_coupling_left, child leg_2_rotY_coupling_left, axis 0.0 1.0 0.0
- added joint leg_2_LCSY_coupling_right: type continuous, parent leg_2_rotX_coupling_right, child leg_2_rotY_coupling_right, axis 0.0 1.0 0.0
- added joint leg_2_LCSZ_coupling_left: type continuous, parent leg_2_rotY_coupling_left, child leg_2_coupling_rod_left, axis 0.0 0.0 1.0
- added joint leg_2_LCSZ_coupling_right: type continuous, parent leg_2_rotY_coupling_right, child leg_2_coupling_rod_right, axis 0.0 0.0 1.0

Commit message: added spherical end joints for easier pybullet constraint formulation

File: src/triped_sim/robot_descriptions/triped.urdf (robot description, URDF)
Before this commit: robot triped, 37 links, 36 joints
Links:
- added link leg_0_rotX_drive_module_left, mass 0
- added link leg_0_rotX_drive_module_right, mass 0
- added link leg_0_rotY_drive_module_left, mass 0
- added link leg_0_rotY_drive_module_right, mass 0
- added link leg_0_rotZ_drive_module_left, mass 0
- added link leg_0_rotZ_drive_module_right, mass 0
- added link leg_1_rotX_drive_module_left, mass 0
- added link leg_1_rotX_drive_module_right, mass 0
- added link leg_1_rotY_drive_module_left, mass 0
- added link leg_1_rotY_drive_module_right, mass 0
- added link leg_1_rotZ_drive_module_left, mass 0
- added link leg_1_rotZ_drive_module_right, mass 0
- added link leg_2_rotX_drive_module_left, mass 0
- added link leg_2_rotX_drive_module_right, mass 0
- added link leg_2_rotY_drive_module_left, mass 0
- added link leg_2_rotY_drive_module_right, mass 0
- added link leg_2_rotZ_drive_module_left, mass 0
- added link leg_2_rotZ_drive_module_right, mass 0
- link leg_0_coupling_rod_left: mass None -> 0
- link leg_0_coupling_rod_right: mass None -> 0
- link leg_0_left: mass None -> 0
- link leg_0_right: mass None -> 0
- link leg_1_coupling_rod_left: mass None -> 0
- link leg_1_coupling_rod_right: mass None -> 0
- link leg_1_left: mass None -> 0
- link leg_1_right: mass None -> 0
- link leg_2_coupling_rod_left: mass None -> 0
- link leg_2_coupling_rod_right: mass None -> 0
- link leg_2_left: mass None -> 0
- link leg_2_right: mass None -> 0
Joints:
- added joint leg_0_LCSX_drive_module_left: type continuous, parent leg_0_coupling_rod_left, child leg_0_rotX_drive_module_left, origin xyz=0.11 0 0 rpy=0.0 0.0 0, axis 1.0 0.0 0.0
- added joint leg_0_LCSX_drive_module_right: type continuous, parent leg_0_right, child leg_0_rotX_drive_module_right, origin xyz=0.085 0 -0.0145 rpy=0.0 0.0 0, axis 1.0 0.0 0.0
- added joint leg_0_LCSY_drive_module_left: type continuous, parent leg_0_rotX_drive_module_left, child leg_0_rotY_drive_module_left, axis 0.0 1.0 0.0
- added joint leg_0_LCSY_drive_module_right: type continuous, parent leg_0_rotX_drive_module_right, child leg_0_rotY_drive_module_right, axis 0.0 1.0 0.0
- added joint leg_0_LCSZ_drive_module_left: type continuous, parent leg_0_rotY_drive_module_left, child leg_0_rotZ_drive_module_left, axis 0.0 0.0 1.0
- added joint leg_0_LCSZ_drive_module_right: type continuous, parent leg_0_rotY_drive_module_right, child leg_0_rotZ_drive_module_right, axis 0.0 0.0 1.0
- added joint leg_1_LCSX_drive_module_left: type continuous, parent leg_1_coupling_rod_left, child leg_1_rotX_drive_module_left, origin xyz=0.11 0 0 rpy=0.0 0.0 0, axis 1.0 0.0 0.0
- added joint leg_1_LCSX_drive_module_right: type continuous, parent leg_1_right, child leg_1_rotX_drive_module_right, origin xyz=0.085 0 -0.0145 rpy=0.0 0.0 0, axis 1.0 0.0 0.0
- added joint leg_1_LCSY_drive_module_left: type continuous, parent leg_1_rotX_drive_module_left, child leg_1_rotY_drive_module_left, axis 0.0 1.0 0.0
- added joint leg_1_LCSY_drive_module_right: type continuous, parent leg_1_rotX_drive_module_right, child leg_1_rotY_drive_module_right, axis 0.0 1.0 0.0
- added joint leg_1_LCSZ_drive_module_left: type continuous, parent leg_1_rotY_drive_module_left, child leg_1_rotZ_drive_module_left, axis 0.0 0.0 1.0
- added joint leg_1_LCSZ_drive_module_right: type continuous, parent leg_1_rotY_drive_module_right, child leg_1_rotZ_drive_module_right, axis 0.0 0.0 1.0
- added joint leg_2_LCSX_drive_module_left: type continuous, parent leg_2_coupling_rod_left, child leg_2_rotX_drive_module_left, origin xyz=0.11 0 0 rpy=0.0 0.0 0, axis 1.0 0.0 0.0
- added joint leg_2_LCSX_drive_module_right: type continuous, parent leg_1_right, child leg_2_rotX_drive_module_right, origin xyz=0.085 0 -0.0145 rpy=0.0 0.0 0, axis 1.0 0.0 0.0
- added joint leg_2_LCSY_drive_module_left: type continuous, parent leg_2_rotX_drive_module_left, child leg_2_rotY_drive_module_left, axis 0.0 1.0 0.0
- added joint leg_2_LCSY_drive_module_right: type continuous, parent leg_2_rotX_drive_module_right, child leg_2_rotY_drive_module_right, axis 0.0 1.0 0.0
- added joint leg_2_LCSZ_drive_module_left: type continuous, parent leg_2_rotY_drive_module_left, child leg_2_rotZ_drive_module_left, axis 0.0 0.0 1.0
- added joint leg_2_LCSZ_drive_module_right: type continuous, parent leg_2_rotY_drive_module_right, child leg_2_rotZ_drive_module_right, axis 0.0 0.0 1.0

Commit message: added collision boxes to urdf

File: src/triped_sim/robot_descriptions/triped.urdf (robot description, URDF)
Before this commit: robot triped, 55 links, 54 joints
Links:
- link leg_0_coupling_rod_left: geometry collision mesh filename=coupling_rod.stl scale=0.001 0.001 0.001; visual mesh filename=coupling_rod.stl scale=0.001 0.001 0.001
- link leg_0_coupling_rod_right: geometry collision mesh filename=coupling_rod.stl scale=0.001 0.001 0.001; visual mesh filename=coupling_rod.stl scale=0.001 0.001 0.001
- link leg_0_drive_module: geometry collision mesh filename=drive_module.stl scale=0.001 0.001 0.001; visual mesh filename=drive_module.stl scale=0.001 0.001 0.001
- link leg_0_left: geometry collision mesh filename=output_lever.stl scale=0.001 0.001 0.001; visual mesh filename=output_lever.stl scale=0.001 0.001 0.001
- link leg_0_right: geometry collision mesh filename=output_lever.stl scale=0.001 0.001 0.001; visual mesh filename=output_lever.stl scale=0.001 0.001 0.001
- link leg_1_coupling_rod_left: geometry collision mesh filename=coupling_rod.stl scale=0.001 0.001 0.001; visual mesh filename=coupling_rod.stl scale=0.001 0.001 0.001
- link leg_1_coupling_rod_right: geometry collision mesh filename=coupling_rod.stl scale=0.001 0.001 0.001; visual mesh filename=coupling_rod.stl scale=0.001 0.001 0.001
- link leg_1_drive_module: geometry collision mesh filename=drive_module.stl scale=0.001 0.001 0.001; visual mesh filename=drive_module.stl scale=0.001 0.001 0.001
- link leg_1_left: geometry collision mesh filename=output_lever.stl scale=0.001 0.001 0.001; visual mesh filename=output_lever.stl scale=0.001 0.001 0.001
- link leg_1_right: geometry collision mesh filename=output_lever.stl scale=0.001 0.001 0.001; visual mesh filename=output_lever.stl scale=0.001 0.001 0.001
- link leg_2_coupling_rod_left: geometry collision mesh filename=coupling_rod.stl scale=0.001 0.001 0.001; visual mesh filename=coupling_rod.stl scale=0.001 0.001 0.001
- link leg_2_coupling_rod_right: geometry collision mesh filename=coupling_rod.stl scale=0.001 0.001 0.001; visual mesh filename=coupling_rod.stl scale=0.001 0.001 0.001
- link leg_2_drive_module: geometry collision mesh filename=drive_module.stl scale=0.001 0.001 0.001; visual mesh filename=drive_module.stl scale=0.001 0.001 0.001
- link leg_2_left: geometry collision mesh filename=output_lever.stl scale=0.001 0.001 0.001; visual mesh filename=output_lever.stl scale=0.001 0.001 0.001
- link leg_2_right: geometry collision mesh filename=output_lever.stl scale=0.001 0.001 0.001; visual mesh filename=output_lever.stl scale=0.001 0.001 0.001

Commit message: changed joint type from continous to revolute

File: src/triped_sim/robot_descriptions/triped.urdf (robot description, URDF)
Before this commit: robot triped, 55 links, 54 joints
Joints:
- joint leg_0_LCSX_coupling_left: limit (none) -> lower=-3.14159265359 upper=3.14159265359 effort=1000.0 velocity=0.5; origin xyz=0.085 0 -0.0145 rpy=0.0 0.0 0 -> xyz=0.085 0 -0.0245 rpy=0.0 0.0 0; type continuous -> revolute
- joint leg_0_LCSX_coupling_right: limit (none) -> lower=-3.14159265359 upper=3.14159265359 effort=1000.0 velocity=0.5; origin xyz=0.085 0 -0.0145 rpy=0.0 0.0 0 -> xyz=0.085 0 -0.0245 rpy=0.0 0.0 0; type continuous -> revolute
- joint leg_0_LCSX_drive_module_left: limit (none) -> lower=-3.14159265359 upper=3.14159265359 effort=1000.0 velocity=0.5; type continuous -> revolute
- joint leg_0_LCSX_drive_module_right: limit (none) -> lower=-3.14159265359 upper=3.14159265359 effort=1000.0 velocity=0.5; origin xyz=0.085 0 -0.0145 rpy=0.0 0.0 0 -> xyz=0.11 0 0 rpy=0.0 0.0 0; type continuous -> revolute
- joint leg_0_LCSY_coupling_left: limit (none) -> lower=-3.14159265359 upper=3.14159265359 effort=1000.0 velocity=0.5; type continuous -> revolute
- joint leg_0_LCSY_coupling_right: limit (none) -> lower=-3.14159265359 upper=3.14159265359 effort=1000.0 velocity=0.5; type continuous -> revolute
- joint leg_0_LCSY_drive_module_left: limit (none) -> lower=-3.14159265359 upper=3.14159265359 effort=1000.0 velocity=0.5; type continuous -> revolute
- joint leg_0_LCSY_drive_module_right: limit (none) -> lower=-3.14159265359 upper=3.14159265359 effort=1000.0 velocity=0.5; type continuous -> revolute
- joint leg_0_LCSZ_coupling_left: limit (none) -> lower=-3.14159265359 upper=3.14159265359 effort=1000.0 velocity=0.5; type continuous -> revolute
- joint leg_0_LCSZ_coupling_right: limit (none) -> lower=-3.14159265359 upper=3.14159265359 effort=1000.0 velocity=0.5; type continuous -> revolute
- joint leg_0_LCSZ_drive_module_left: limit (none) -> lower=-3.14159265359 upper=3.14159265359 effort=1000.0 velocity=0.5; type continuous -> revolute
- joint leg_0_LCSZ_drive_module_right: limit (none) -> lower=-3.14159265359 upper=3.14159265359 effort=1000.0 velocity=0.5; type continuous -> revolute
- joint leg_1_LCSX_coupling_left: limit (none) -> lower=-3.14159265359 upper=3.14159265359 effort=1000.0 velocity=0.5; origin xyz=0.085 0 -0.0145 rpy=0.0 0.0 0 -> xyz=0.085 0 -0.0245 rpy=0.0 0.0 0; type continuous -> revolute
- joint leg_1_LCSX_coupling_right: limit (none) -> lower=-3.14159265359 upper=3.14159265359 effort=1000.0 velocity=0.5; origin xyz=0.085 0 -0.0145 rpy=0.0 0.0 0 -> xyz=0.085 0 -0.0245 rpy=0.0 0.0 0; type continuous -> revolute
- joint leg_1_LCSX_drive_module_left: limit (none) -> lower=-3.14159265359 upper=3.14159265359 effort=1000.0 velocity=0.5; type continuous -> revolute
- joint leg_1_LCSX_drive_module_right: limit (none) -> lower=-3.14159265359 upper=3.14159265359 effort=1000.0 velocity=0.5; origin xyz=0.085 0 -0.0145 rpy=0.0 0.0 0 -> xyz=0.11 0 0 rpy=0.0 0.0 0; type continuous -> revolute
- joint leg_1_LCSY_coupling_left: limit (none) -> lower=-3.14159265359 upper=3.14159265359 effort=1000.0 velocity=0.5; type continuous -> revolute
- joint leg_1_LCSY_coupling_right: limit (none) -> lower=-3.14159265359 upper=3.14159265359 effort=1000.0 velocity=0.5; type continuous -> revolute
- joint leg_1_LCSY_drive_module_left: limit (none) -> lower=-3.14159265359 upper=3.14159265359 effort=1000.0 velocity=0.5; type continuous -> revolute
- joint leg_1_LCSY_drive_module_right: limit (none) -> lower=-3.14159265359 upper=3.14159265359 effort=1000.0 velocity=0.5; type continuous -> revolute
- joint leg_1_LCSZ_coupling_left: limit (none) -> lower=-3.14159265359 upper=3.14159265359 effort=1000.0 velocity=0.5; type continuous -> revolute
- joint leg_1_LCSZ_coupling_right: limit (none) -> lower=-3.14159265359 upper=3.14159265359 effort=1000.0 velocity=0.5; type continuous -> revolute
- joint leg_1_LCSZ_drive_module_left: limit (none) -> lower=-3.14159265359 upper=3.14159265359 effort=1000.0 velocity=0.5; type continuous -> revolute
- joint leg_1_LCSZ_drive_module_right: limit (none) -> lower=-3.14159265359 upper=3.14159265359 effort=1000.0 velocity=0.5; type continuous -> revolute
- joint leg_2_LCSX_coupling_left: limit (none) -> lower=-3.14159265359 upper=3.14159265359 effort=1000.0 velocity=0.5; origin xyz=0.085 0 -0.0145 rpy=0.0 0.0 0 -> xyz=0.085 0 -0.0245 rpy=0.0 0.0 0; type continuous -> revolute
- joint leg_2_LCSX_coupling_right: limit (none) -> lower=-3.14159265359 upper=3.14159265359 effort=1000.0 velocity=0.5; origin xyz=0.085 0 -0.0145 rpy=0.0 0.0 0 -> xyz=0.085 0 -0.0245 rpy=0.0 0.0 0; type continuous -> revolute
- joint leg_2_LCSX_drive_module_left: limit (none) -> lower=-3.14159265359 upper=3.14159265359 effort=1000.0 velocity=0.5; type continuous -> revolute
- joint leg_2_LCSX_drive_module_right: limit (none) -> lower=-3.14159265359 upper=3.14159265359 effort=1000.0 velocity=0.5; origin xyz=0.085 0 -0.0145 rpy=0.0 0.0 0 -> xyz=0.11 0 0 rpy=0.0 0.0 0; type continuous -> revolute
- joint leg_2_LCSY_coupling_left: limit (none) -> lower=-3.14159265359 upper=3.14159265359 effort=1000.0 velocity=0.5; type continuous -> revolute
- joint leg_2_LCSY_coupling_right: limit (none) -> lower=-3.14159265359 upper=3.14159265359 effort=1000.0 velocity=0.5; type continuous -> revolute
- joint leg_2_LCSY_drive_module_left: limit (none) -> lower=-3.14159265359 upper=3.14159265359 effort=1000.0 velocity=0.5; type continuous -> revolute
- joint leg_2_LCSY_drive_module_right: limit (none) -> lower=-3.14159265359 upper=3.14159265359 effort=1000.0 velocity=0.5; type continuous -> revolute
- joint leg_2_LCSZ_coupling_left: limit (none) -> lower=-3.14159265359 upper=3.14159265359 effort=1000.0 velocity=0.5; type continuous -> revolute
- joint leg_2_LCSZ_coupling_right: limit (none) -> lower=-3.14159265359 upper=3.14159265359 effort=1000.0 velocity=0.5; type continuous -> revolute
- joint leg_2_LCSZ_drive_module_left: limit (none) -> lower=-3.14159265359 upper=3.14159265359 effort=1000.0 velocity=0.5; type continuous -> revolute
- joint leg_2_LCSZ_drive_module_right: limit (none) -> lower=-3.14159265359 upper=3.14159265359 effort=1000.0 velocity=0.5; type continuous -> revolute

Commit message: added small maß to swing leg assembly

File: src/triped_sim/robot_descriptions/triped.urdf (robot description, URDF)
Before this commit: robot triped, 55 links, 54 joints
Links:
- link leg_0_coupling_rod_left: mass 0 -> 0.01
- link leg_0_coupling_rod_right: mass 0 -> 0.01
- link leg_0_left: mass 0 -> 0.01
- link leg_0_right: mass 0 -> 0.01
- link leg_0_rotX: mass 0 -> 0.01
- link leg_0_rotX_coupling_left: mass 0 -> 0.01
- link leg_0_rotX_coupling_right: mass 0 -> 0.01
- link leg_0_rotX_drive_module_left: mass 0 -> 0.01
- link leg_0_rotX_drive_module_right: mass 0 -> 0.01
- link leg_0_rotY: mass 0 -> 0.01
- link leg_0_rotY_coupling_left: mass 0 -> 0.01
- link leg_0_rotY_coupling_right: mass 0 -> 0.01
- link leg_0_rotY_drive_module_left: mass 0 -> 0.01
- link leg_0_rotY_drive_module_right: mass 0 -> 0.01
- link leg_0_rotZ_drive_module_left: mass 0 -> 0.01
- link leg_0_rotZ_drive_module_right: mass 0 -> 0.01
- link leg_1_coupling_rod_left: mass 0 -> 0.01
- link leg_1_coupling_rod_right: mass 0 -> 0.01
- link leg_1_left: mass 0 -> 0.01
- link leg_1_right: mass 0 -> 0.01
- link leg_1_rotX: mass 0 -> 0.01
- link leg_1_rotX_coupling_left: mass 0 -> 0.01
- link leg_1_rotX_coupling_right: mass 0 -> 0.01
- link leg_1_rotX_drive_module_left: mass 0 -> 0.01
- link leg_1_rotX_drive_module_right: mass 0 -> 0.01
- link leg_1_rotY: mass 0 -> 0.01
- link leg_1_rotY_coupling_left: mass 0 -> 0.01
- link leg_1_rotY_coupling_right: mass 0 -> 0.01
- link leg_1_rotY_drive_module_left: mass 0 -> 0.01
- link leg_1_rotY_drive_module_right: mass 0 -> 0.01
- link leg_1_rotZ_drive_module_left: mass 0 -> 0.01
- link leg_1_rotZ_drive_module_right: mass 0 -> 0.01
- link leg_2_coupling_rod_left: mass 0 -> 0.01
- link leg_2_coupling_rod_right: mass 0 -> 0.01
- link leg_2_left: mass 0 -> 0.01
- link leg_2_right: mass 0 -> 0.01
- link leg_2_rotX: mass 0 -> 0.01
- link leg_2_rotX_coupling_left: mass 0 -> 0.01
- link leg_2_rotX_coupling_right: mass 0 -> 0.01
- link leg_2_rotX_drive_module_left: mass 0 -> 0.01
- link leg_2_rotX_drive_module_right: mass 0 -> 0.01
- link leg_2_rotY: mass 0 -> 0.01
- link leg_2_rotY_coupling_left: mass 0 -> 0.01
- link leg_2_rotY_coupling_right: mass 0 -> 0.01
- link leg_2_rotY_drive_module_left: mass 0 -> 0.01
- link leg_2_rotY_drive_module_right: mass 0 -> 0.01
- link leg_2_rotZ_drive_module_left: mass 0 -> 0.01
- link leg_2_rotZ_drive_module_right: mass 0 -> 0.01

Commit message: fixed coupling rods for leg 2

File: src/triped_sim/robot_descriptions/triped.urdf (robot description, URDF)
Before this commit: robot triped, 55 links, 54 joints
Joints:
- joint leg_2_LCSX_coupling_left: parent leg_1_left -> leg_2_left
- joint leg_2_LCSX_coupling_right: parent leg_1_right -> leg_2_right
- joint leg_2_LCSX_drive_module_right: parent leg_1_right -> leg_2_right
