Commit message: fixed left subchain constraint

File: src/triped_sim/robot_descriptions/triped.urdf (robot description, URDF)
Before this commit: robot triped, 55 links, 54 joints
Joints:
- joint leg_0_LCSX_coupling_left: limit lower=-3.14159265359 upper=3.14159265359 effort=1000.0 velocity=0.5 -> (none); type revolute -> continuous
- joint leg_0_LCSX_coupling_right: limit lower=-3.14159265359 upper=3.14159265359 effort=1000.0 velocity=0.5 -> (none); type revolute -> continuous
- joint leg_0_LCSX_drive_module_left: limit lower=-3.14159265359 upper=3.14159265359 effort=1000.0 velocity=0.5 -> (none); type revolute -> continuous
- joint leg_0_LCSX_drive_module_right: limit lower=-3.14159265359 upper=3.14159265359 effort=1000.0 velocity=0.5 -> (none); type revolute -> continuous
- joint leg_0_LCSY_coupling_left: limit lower=-3.14159265359 upper=3.14159265359 effort=1000.0 velocity=0.5 -> (none); type revolute -> continuous
- joint leg_0_LCSY_coupling_right: limit lower=-3.14159265359 upper=3.14159265359 effort=1000.0 velocity=0.5 -> (none); type revolute -> continuous
- joint leg_0_LCSY_drive_module_left: limit lower=-3.14159265359 upper=3.14159265359 effort=1000.0 velocity=0.5 -> (none); type revolute -> continuous
- joint leg_0_LCSY_drive_module_right: limit lower=-3.14159265359 upper=3.14159265359 effort=1000.0 velocity=0.5 -> (none); type revolute -> continuous
- joint leg_0_LCSZ_coupling_left: limit lower=-3.14159265359 upper=3.14159265359 effort=1000.0 velocity=0.5 -> (none); type revolute -> continuous
- joint leg_0_LCSZ_coupling_right: limit lower=-3.14159265359 upper=3.14159265359 effort=1000.0 velocity=0.5 -> (none); type revolute -> continuous
- joint leg_0_LCSZ_drive_module_left: limit lower=-3.14159265359 upper=3.14159265359 effort=1000.0 velocity=0.5 -> (none); type revolute -> continuous
- joint leg_0_LCSZ_drive_module_right: limit lower=-3.14159265359 upper=3.14159265359 effort=1000.0 velocity=0.5 -> (none); type revolute -> continuous
- joint leg_1_LCSX_coupling_left: limit lower=-3.14159265359 upper=3.14159265359 effort=1000.0 velocity=0.5 -> (none); type revolute -> continuous
- joint leg_1_LCSX_coupling_right: limit lower=-3.14159265359 upper=3.14159265359 effort=1000.0 velocity=0.5 -> (none); type revolute -> continuous
- joint leg_1_LCSX_drive_module_left: limit lower=-3.14159265359 upper=3.14159265359 effort=1000.0 velocity=0.5 -> (none); type revolute -> continuous
- joint leg_1_LCSX_drive_module_right: limit lower=-3.14159265359 upper=3.14159265359 effort=1000.0 velocity=0.5 -> (none); type revolute -> continuous
- joint leg_1_LCSY_coupling_left: limit lower=-3.14159265359 upper=3.14159265359 effort=1000.0 velocity=0.5 -> (none); type revolute -> continuous
- joint leg_1_LCSY_coupling_right: limit lower=-3.14159265359 upper=3.14159265359 effort=1000.0 velocity=0.5 -> (none); type revolute -> continuous
- joint leg_1_LCSY_drive_module_left: limit lower=-3.14159265359 upper=3.14159265359 effort=1000.0 velocity=0.5 -> (none); type revolute -> continuous
- joint leg_1_LCSY_drive_module_right: limit lower=-3.14159265359 upper=3.14159265359 effort=1000.0 velocity=0.5 -> (none); type revolute -> continuous
- joint leg_1_LCSZ_coupling_left: limit lower=-3.14159265359 upper=3.14159265359 effort=1000.0 velocity=0.5 -> (none); type revolute -> continuous
- joint leg_1_LCSZ_coupling_right: limit lower=-3.14159265359 upper=3.14159265359 effort=1000.0 velocity=0.5 -> (none); type revolute -> continuous
- joint leg_1_LCSZ_drive_module_left: limit lower=-3.14159265359 upper=3.14159265359 effort=1000.0 velocity=0.5 -> (none); type revolute -> continuous
- joint leg_1_LCSZ_drive_module_right: limit lower=-3.14159265359 upper=3.14159265359 effort=1000.0 velocity=0.5 -> (none); type revolute -> continuous
- joint leg_2_LCSX_coupling_left: limit lower=-3.14159265359 upper=3.14159265359 effort=1000.0 velocity=0.5 -> (none); type revolute -> continuous
- joint leg_2_LCSX_coupling_right: limit lower=-3.14159265359 upper=3.14159265359 effort=1000.0 velocity=0.5 -> (none); type revolute -> continuous
- joint leg_2_LCSX_drive_module_left: limit lower=-3.14159265359 upper=3.14159265359 effort=1000.0 velocity=0.5 -> (none); type revolute -> continuous
- joint leg_2_LCSX_drive_module_right: limit lower=-3.14159265359 upper=3.14159265359 effort=1000.0 velocity=0.5 -> (none); type revolute -> continuous
- joint leg_2_LCSY_coupling_left: limit lower=-3.14159265359 upper=3.14159265359 effort=1000.0 velocity=0.5 -> (none); type revolute -> continuous
- joint leg_2_LCSY_coupling_right: limit lower=-3.14159265359 upper=3.14159265359 effort=1000.0 velocity=0.5 -> (none); type revolute -> continuous
- joint leg_2_LCSY_drive_module_left: limit lower=-3.14159265359 upper=3.14159265359 effort=1000.0 velocity=0.5 -> (none); type revolute -> continuous
- joint leg_2_LCSY_drive_module_right: limit lower=-3.14159265359 upper=3.14159265359 effort=1000.0 velocity=0.5 -> (none); type revolute -> continuous
- joint leg_2_LCSZ_coupling_left: limit lower=-3.14159265359 upper=3.14159265359 effort=1000.0 velocity=0.5 -> (none); type revolute -> continuous
- joint leg_2_LCSZ_coupling_right: limit lower=-3.14159265359 upper=3.14159265359 effort=1000.0 velocity=0.5 -> (none); type revolute -> continuous
- joint leg_2_LCSZ_drive_module_left: limit lower=-3.14159265359 upper=3.14159265359 effort=1000.0 velocity=0.5 -> (none); type revolute -> continuous
- joint leg_2_LCSZ_drive_module_right: limit lower=-3.14159265359 upper=3.14159265359 effort=1000.0 velocity=0.5 -> (none); type revolute -> continuous

Commit message: fixed right subchain urdf

File: src/triped_sim/robot_descriptions/triped.urdf (robot description, URDF)
Before this commit: robot triped, 55 links, 54 joints
Joints:
- joint leg_0_LCSX_drive_module_right: parent leg_0_right -> leg_0_coupling_rod_right
- joint leg_1_LCSX_drive_module_right: parent leg_1_right -> leg_1_coupling_rod_right
- joint leg_2_LCSX_drive_module_right: parent leg_2_right -> leg_2_coupling_rod_right

Commit message: made joint names compliant with trip_kinematics conventions

File: src/triped_sim/robot_descriptions/triped.urdf (robot description, URDF)
Before this commit: robot triped, 55 links, 54 joints
Joints:
- removed joint leg_0/extend/joint
- removed joint leg_0/swing/left/joint
- removed joint leg_0/swing/right/joint
- removed joint leg_1/extend/joint
- removed joint leg_1/swing/left/joint
- removed joint leg_1/swing/right/joint
- removed joint leg_2/extend/joint
- removed joint leg_2/swing/left/joint
- removed joint leg_2/swing/right/joint
- added joint leg_0_extend_joint_ry: type revolute, parent leg_0_drive_module, child leg_0_open, origin xyz=1.640 0.0 -0.037 rpy=0.0 -0.05235987756 0.0, axis 0.0 1.0 0.0, limit lower=-0.48869219055 upper=0.0034906585 effort=1000.0 velocity=0.5
- added joint leg_0_swing_left: type revolute, parent chassis, child leg_0_left, origin xyz=0.1398076694471282 -0.054999840697609804 -0.051 rpy=0.0 0.0 -0.37480073021952226, axis 0.0 0.0 1.0, limit lower=-1.57079632679 upper=1.57079632679 effort=1000.0 velocity=0.5
- added joint leg_0_swing_right: type revolute, parent chassis, child leg_0_right, origin xyz=0.1398076694471282 0.054999840697609804 -0.051 rpy=0.0 0.0 0.37480073021952226, axis 0.0 0.0 1.0, limit lower=-1.57079632679 upper=1.57079632679 effort=1000.0 velocity=0.5
- added joint leg_1_extend_joint_ry: type revolute, parent leg_1_drive_module, child leg_1_open, origin xyz=1.640 0.0 -0.037 rpy=0.0 -0.05235987756 0.0, axis 0.0 1.0 0.0, limit lower=-0.48869219055 upper=0.0034906585 effort=1000.0 velocity=0.5
- added joint leg_1_swing_left: type revolute, parent chassis, child leg_1_left, origin xyz=-0.11753509397179145 -0.0935770730363056 -0.051 rpy=0.0 0.0 -2.469195832612718, axis 0.0 0.0 1.0, limit lower=-1.57079632679 upper=1.57079632679 effort=1000.0 velocity=0.5
- added joint leg_1_swing_right: type revolute, parent chassis, child leg_1_right, origin xyz=-0.022272575475336735 -0.14857691373391543 -0.051 rpy=0.0 0.0 -1.719594372173673, axis 0.0 0.0 1.0, limit lower=-1.57079632679 upper=1.57079632679 effort=1000.0 velocity=0.5
- added joint leg_2_extend_joint_ry: type revolute, parent leg_2_drive_module, child leg_2_open, origin xyz=1.640 0.0 -0.037 rpy=0.0 -0.05235987756 0.0, axis 0.0 1.0 0.0, limit lower=-0.48869219055 upper=0.0034906585 effort=1000.0 velocity=0.5
- added joint leg_2_swing_left: type revolute, parent chassis, child leg_2_left, origin xyz=-0.022272575475336905 0.1485769137339154 -0.051 rpy=0.0 0.0 -4.563590935005912, axis 0.0 0.0 1.0, limit lower=-1.57079632679 upper=1.57079632679 effort=1000.0 velocity=0.5
- added joint leg_2_swing_right: type revolute, parent chassis, child leg_2_right, origin xyz=-0.11753509397179142 0.09357707303630562 -0.051 rpy=0.0 0.0 -3.8139894745668688, axis 0.0 0.0 1.0, limit lower=-1.57079632679 upper=1.57079632679 effort=1000.0 velocity=0.5
